File: doc/Clock_1.sch (EAGLE design)
At the start: 175 parts, among them IC2 MCP23017, IC3 MCP604SL, IC8 LM1117-3.3, Q1 BC846, Q2 BC846, Q3 BC846, Q4 BC846, Q5 BC846, Q6 BC846, Q7 BC846, U1 RP2040, U2 MCP6002_, Y1 12MHz

Commit message: need to update screenshots. need to handle PORTB
Parts:
- removed C33, C55: 10uF, rcl:CPOL-EUB
- removed C35, C40, C44, C45, C46, C47, C48, C49, C50, C51: 100n, rcl:C-EUC0603
- removed C42, C43: 2.2uF, rcl:C-EUC0603
- removed D30: SS1040_R1_00001, diode:DIODE-SOD123
- removed IC2: MCP23017, adafruit:MCP23017
- removed IC3: MCP604SL, linear:MCP604SL
- removed PL1: (no value), jt-con-tyco:2X5-1241050
- removed R21, R58, R70: 1k, rcl:R-EU_R0603
- removed R54, R55: 27 Ohm, rcl:R-EU_R0603
- removed SW1: (no value), adafruit:SWITCH_PUSHBUTTONSOFTTOUCHSMD_SJ
- removed Y1: 12MHz, SparkFun-Clocks:CRYSTAL-25MHZ-WE-SMD-2.0X1.6MM-WE
- added C101, C103, C107, C110, C112, C113, C114, C117, C118, C120, C121, C122: 100n, rcl:C-EUC0603
- added C109, C111: 10uF, rcl:CPOL-EUB
- added D3: SS1040_R1_00001, diode:DIODE-SOD123
- added IC101: MCP23017SS, adafruit:MCP23017SS
- added J1: (no value), SparkFun-Connectors:CONN_05X2RA
- added JP100, JP2: (no value), pinhead:PINHD-1X151X15ç
- added JP101, JP3: (no value), pinhead:PINHD-1X81X8ç
- added JP102, JP4: (no value), pinhead:PINHD-1X12Ç
- added R114: 100k, rcl:R-EU_R0603
- added R115: 33k, rcl:R-EU_R0603
- added R143, R144: 1k, rcl:R-EU_R0603
- added R147: 560 Ohm, rcl:R-EU_R0603
- added SW5: (no value), switch-omron:10-XX
- added U101, U102: MCP6002_, MTM:MCP6002_
- added Y2: 12MHZ, microbuilder:CRYSTAL2.5X2.0
- +*-, ALT, CHANCE, CV, MUTE, PRESET, TEMPO: value BUTTON_NEOPIXEL -> BUTTON_NEOPIXELBUTTON_PIXEL_ç; device switch-tact:BUTTON_NEOPIXEL -> switch-tact:BUTTON_NEOPIXELBUTTON_PIXEL_ç
- C1, C5: value 100n -> 10uF; device rcl:C-EUC0603 -> rcl:CPOL-EUB
- C10: value 22uF -> 100n
- C11, C18: value 10uF -> 100n; device rcl:CPOL-EUB -> rcl:C-EUC0603
- C12: value 2.2uF -> 22uF
- C13: value 2.2uF -> 10uF; device rcl:C-EUC0603 -> rcl:CPOL-EUB
- C14, C19, C21: value 100n -> 2.2uF
- C2: value 10uF -> 10n; device rcl:CPOL-EUB -> rcl:C-EUC0603
- C20: value 10uF -> 2.2uF; device rcl:CPOL-EUB -> rcl:C-EUC0603
- C28, C29: value 100n -> 22pF
- C3: value 10n -> 100n
- C6: device rcl:C-EUC0603 -> rcl:CPOL-EUB
- C7: value 100n -> 10uF
- F1: value F1 -> F2
- F2: value F2 -> F1
- L1: value 4.7uH -> 0.1uH
- L3: value 0.1uH -> 4.7uH
- PLAY: value DTS-6_LEDTME -> DTS-6_LED; device switch-tact:DTS-6_LEDTME -> switch-tact:DTS-6_LED
- POWER: value M05X2SHD_LOCK -> M05X2RAF; device SparkFun:M05X2SHD_LOCK -> SparkFun:M05X2RAF
- R10: value 33k -> 1k
- R5: value 1M -> 10k
- R6: value 10k -> 1k
- R7: value 1k -> 1M
- R8: value 100k -> 27 Ohm
- R9: value 560 Ohm -> 27 Ohm
- U$1: value W25Q128JVSIQ -> BL9342; device SparkFun-IC-Memory:W25Q128JVSIQ -> adafruit:BL9342
- U$2: value BL9342 -> W25Q128JVSIQ; device adafruit:BL9342 -> SparkFun-IC-Memory:W25Q128JVSIQ
- renumbered C30 to C119, C31 to C116, C32 to C115, C34 to C105, C36 to C102, C37 to C104, C38 to C106, C39 to C108, C41 to C100, D21 to D2, IC8 to IC100, Q1 to Q101, Q2 to Q100, Q3 to Q102, Q4 to Q103, Q5 to Q104, Q6 to Q105, Q7 to Q106, R11 to R148, R12 to R117, R13 to R126, R14 to R135, R15 to R142, R16 to R111, R17 to R116, R18 to R113, R19 to R112, R20 to R146, R22 to R127, R23 to R125, R24 to R128, R25 to R124, R26 to R129, R27 to R123, R28 to R121, R29 to R132, R30 to R139, R31 to R140, R32 to R105, R33 to R100, R34 to R104, R35 to R107, R36 to R101, R37 to R150, R38 to R149, R39 to R145, R40 to R120, R41 to R108, R42 to R103, R43 to R122, R44 to R118, R45 to R119, R46 to R130, R47 to R134, R48 to R133, R49 to R131, R50 to R138, R51 to R141, R52 to R137, R53 to R136, R57 to R106, R67 to R102, R72 to R110, U$3 to U$100, U2 to U100
Connections:
- removed net +*-: +*-.1, +*-.3, U1.GPIO12
- removed net A: A.3, A.4, U1.GPIO15
- removed net ALT: ALT.1, ALT.3, U1.GPIO8
- removed net A_OUT: LED_A_OUT.C, R111.2, U1.GPIO24
- removed net B: B.3, B.4, U1.GPIO16
- removed net B_OUT: LED_B_OUT.C, R120.2, U1.GPIO25
- removed net C: C.3, C.4, U1.GPIO17
- removed net CHAN: CHANCE.1, CHANCE.3, U1.GPIO10
- removed net CV: CV.1, CV.3, U1.GPIO9
- removed net C_OUT: LED_C_OUT.C, R130.2, U1.GPIO26/ADC0
- removed net D: D.3, D.4, U1.GPIO18
- removed net D_OUT: LED_D_OUT.C, R138.2, U1.GPIO27/ADC1
- removed net ENC_A: C116.1, R150.1, U1.GPIO2
- removed net ENC_B: C115.2, R146.2, U1.GPIO3
- removed net ENC_SW: ENCODERB.E, U1.GPIO4
- removed net I2C0_SCL: IC2.SCL, U1.GPIO1
- removed net I2C0_SDA: IC2.SDA, U1.GPIO0
- removed net I2C1_SCL: R128.2, U$100.SCL
- removed net I2C1_SDA: R124.2, U$100.SDA
- removed net LA: A.P$1, IC2.GPB7
- removed net LB: B.P$1, U1.GPIO20
- removed net LC: C.P$1, U1.GPIO21
- removed net LD: D.P$1, U1.GPIO22
- removed net MUTE: MUTE.1, MUTE.3, U1.GPIO13
- removed net N$70: BEAT.C, IC2.GPB5
- removed net N$90: C12.1, U1.LDO_OUT
- removed net NEO: R9.1, U1.GPIO7
- removed net PLAY: PLAY.3, PLAY.4, U1.GPIO19
- removed net PRESE_CV: C100.2, R107.1, U1.GPIO29/ADC3, U100A.OUT
- removed net PREST: PRESET.1, PRESET.3, U1.GPIO14
- removed net RESE_CV: Q101.C, R108.1, U1.GPIO6
- removed net ST/SP: R58.2, U1.GPIO23
- removed net SYNC_CV: Q102.C, R110.1, U1.GPIO5
- removed net TEMP: TEMPO.1, TEMPO.3, U1.GPIO11
- new net +*-_B: JP4.1, U1.GPIO12
- new net +*-_T: +*-.1, +*-.3, JP102.1
- new net ALT_B: JP2.12, U1.GPIO11
- new net ALT_T: ALT.1, ALT.3, JP100.12
- new net A_B: JP2.2, U1.GPIO1
- new net A_OUT_B: JP3.3, U1.GPIO28/ADC2
- new net A_OUT_T: JP101.3, LED_A_OUT.C, R111.2
- new net A_T: A.3, A.4, JP100.2
- new net B_B: JP2.4, U1.GPIO3
- new net B_OUT_B: JP3.4, U1.GPIO27/ADC1
- new net B_OUT_T: JP101.4, LED_B_OUT.C, R120.2
- new net B_T: B.3, B.4, JP100.4
- new net CHAN_B: JP4.10, U1.GPIO22
- new net CHAN_T: CHANCE.1, CHANCE.3, JP102.10
- new net CV_B: JP4.2, U1.GPIO13
- new net CV_T: CV.1, CV.3, JP102.2
- new net C_B: JP2.8, U1.GPIO7
- new net C_OUT_B: JP3.6, U1.GPIO26/ADC0
- new net C_OUT_T: JP101.6, LED_C_OUT.C, R130.2
- new net C_T: C.3, C.4, JP100.8
- new net D_B: JP2.6, U1.GPIO5
- new net D_OUT_B: JP3.7, U1.GPIO25
- new net D_OUT_T: JP101.7, LED_D_OUT.C, R138.2
- new net D_T: D.3, D.4, JP100.6
- new net ENC_A_B: JP4.5, U1.GPIO18
- new net ENC_A_T: C116.1, JP102.5, R150.1
- new net ENC_B_B: JP4.6, U1.GPIO19
- new net ENC_B_T: C115.2, JP102.6, R146.2
- new net ENC_SW_B: JP4.11, U1.GPIO23
- new net ENC_SW_T: ENCODERB.E, JP102.11
- new net I2C0_SCL_B: JP3.2, U1.GPIO17
- new net I2C0_SCL_T: IC101.SCL, JP101.2, R128.2, U$100.SCL
- new net I2C0_SDA_B: JP3.1, U1.GPIO16
- new net I2C0_SDA_T: IC101.SDA, JP101.1, R124.2, U$100.SDA
- new net LA_B: JP2.1, U1.GPIO0
- new net LA_T: A.P$1, JP100.1
- new net LB_B: JP2.3, U1.GPIO2
- new net LB_T: B.P$1, JP100.3
- new net LC_B: JP2.5, U1.GPIO4
- new net LC_T: C.P$1, JP100.5
- new net LD_B: JP2.7, U1.GPIO6
- new net LD_T: D.P$1, JP100.7
- new net MUTE_B: JP4.3, U1.GPIO14
- new net MUTE_T: JP102.3, MUTE.1, MUTE.3
- new net N$13: BAR.A, IC101.GPB4
- new net NEO_B: JP2.9, U1.GPIO8
- new net NEO_T: JP100.9, R147.1
- new net PLAY_B: JP4.9, U1.GPIO21
- new net PLAY_T: JP102.9, PLAY.3, PLAY.4
- new net PRESE_CV_B: JP4.8, U1.GPIO29/ADC3
- new net PRESE_CV_T: C100.2, JP102.8, R107.1, U100A.OUT
- new net PREST_B: JP4.7, U1.GPIO20
- new net PREST_T: JP102.7, PRESET.1, PRESET.3
- new net RESE_CV_B: JP2.11, U1.GPIO10
- new net RESE_CV_T: JP100.11, Q101.C, R108.1
- new net ST/SP_B: JP4.4, U1.GPIO15
- new net ST/SP_T: JP102.4, R109.2
- new net SYNC_CV_B: JP2.10, U1.GPIO9
- new net SYNC_CV_T: JP100.10, Q102.C, R110.1
- new net TEMP_B: JP4.12, U1.GPIO24
- new net TEMP_T: JP102.12, TEMPO.1, TEMPO.3
- net +12V: now also C1.+, C109.+, C110.1, C6.+, C8.1, JP101.5, JP3.5, L1.1; no longer C18.+, C19.1, C2.+, C33.+, C35.1, L2.1
- net +3V3: now also C101.1, C103.1, C107.1, C111.+, C112.1, C113.1, C114.1, C117.1, C118.1, C120.1, C121.1, C122.1, IC101.!RESET, IC101.VDD, U101P.V+, U102P.V+; no longer C20.+, C21.1, C22.1, C23.1, C24.1, C25.1, C26.1, C27.1, C28.1, C29.1, C40.1, IC2.!RESET, IC2.VDD, IC3P.V+, R21.1, R70.1
- net -12V: now also C4.2, C5.-, D1.A; no longer C50.2, C55.-, D30.A
- net A_CV: now also R115.1, U101A.OUT; no longer IC3B.OUT, R10.1
- net B_CV: now also U101B.OUT; no longer IC3A.OUT
- net C_CV: now also U102A.OUT; no longer IC3C.OUT
- net D_CV: now also U102B.OUT; no longer IC3D.OUT
- net GND: now also C1.-, C101.2, C103.2, C107.2, C109.-, C110.2, C111.-, C112.2, C113.2, C114.2, C117.2, C118.2, C12.1, C120.2, C121.2, C122.2, C13.-, C14.2, C15.2, C17.1, C18.1, C2.2, C20.2, C22.1, C23.1, C24.1, C25.1, C26.1, C27.1, C28.1, C5.+, C6.-, C8.2, C9.2, D3.A, IC101.A0, IC101.A1, IC101.A2, IC101.VSS, J1.3, J1.5, J1.9, JP100.13, JP100.14, JP100.15, JP101.8, JP2.13, JP2.14, JP2.15, JP3.8, R143.1, R144.1, R7.1, SW5.P, SW5.P1, U101A.+IN, U101B.+IN, U101P.V-, U102A.+IN, U102B.+IN, U102P.V-; no longer C1.2, C10.1, C11.-, C12.2, C13.2, C14.1, C15.1, C17.2, C18.-, C2.-, C20.-, C22.2, C23.2, C24.2, C25.2, C26.2, C27.2, C28.2, C33.-, C35.2, C40.2, C42.2, C43.2, C44.1, C45.1, C46.1, C47.1, C48.1, C49.1, C5.2, C50.1, C51.1, C55.+, C6.2, D1.A, IC2.A0, IC2.A1, IC2.A2, IC2.VSS, IC3A.+IN, IC3B.+IN, IC3C.+IN, IC3D.+IN, IC3P.V-, PL1.3, PL1.5, PL1.9, R5.1, SW1.P$1, Y1.GND
- net LPLAY: now also IC101.GPB6; no longer IC2.GPB6
- net MEM_CLK: now also U$2.SCK; no longer U$1.SCK
- net MEM_CS: now also R5.1, U$2.CS; no longer R7.1, U$1.CS
- net MEM_I00: now also U$2.DI; no longer U$1.DI
- net MEM_I01: now also U$2.D0; no longer U$1.D0
- net MEM_I02: now also U$2.I02; no longer U$1.I02
- net MEM_I03: now also U$2.I03; no longer U$1.I03
- net N$1: now also R10.2; no longer R109.2
- net N$10: now also C11.2, C12.2, L3.2; no longer C10.2, C9.2, L1.2
- net N$11: now also IC101.GPA0; no longer IC2.GPA0
- net N$12: now also R8.2; no longer R55.2
- net N$14: now also R9.1; no longer R54.1
- net N$15: now also R7.2; no longer R5.2
- net N$16: now also IC101.GPA1; no longer IC2.GPA1
- net N$17: now also R6.2, SW5.S, SW5.S1; no longer R7.2, SW1.P$2
- net N$18: now also IC101.GPA2; no longer IC2.GPA2
- net N$19: now also IC101.GPA3; no longer IC2.GPA3
- net N$2: now also C28.2, Y2.2; no longer C4.2, Y1.1
- net N$20: now also IC101.GPA4; no longer IC2.GPA4
- net N$21: now also IC101.GPA5; no longer IC2.GPA5
- net N$22: now also IC101.GPA6; no longer IC2.GPA6
- net N$23: now also IC101.GPA7; no longer IC2.GPA7
- net N$24: now also IC101.GPB0; no longer IC2.GPB0
- net N$25: now also IC101.GPB1; no longer IC2.GPB1
- net N$26: now also IC101.GPB2; no longer IC2.GPB2
- net N$27: now also IC101.GPB3; no longer IC2.GPB3
- net N$28: now also R114.1, R115.2, U101A.-IN; no longer IC3B.-IN, R10.2, R8.1
- net N$29: now also R147.2; no longer R9.2
- net N$3: now also C29.1, R10.1, Y2.1; no longer C1.1, R109.1, Y1.2
- net N$31: now also PRESET.DI; no longer CHANCE.DI
- net N$32: now also PRESET.DO; no longer CHANCE.DO
- net N$33: now also CHANCE.DI; no longer +*-.DI
- net N$34: now also CHANCE.DO; no longer +*-.DO
- net N$35: now also +*-.DI; no longer PRESET.DI
- net N$37: now also U101B.-IN; no longer IC3A.-IN
- net N$38: now also U102A.-IN; no longer IC3C.-IN
- net N$39: now also U102B.-IN; no longer IC3D.-IN
- net N$4: now also U$1.EN; no longer U$2.EN
- net N$43: now also F2.2; no longer F1.2
- net N$44: now also F2.1; no longer F1.1
- net N$45: now also F1.2; no longer F2.2
- net N$46: now also D1.C, F1.1; no longer D30.C, F2.1
- net N$5: now also C3.1, C9.1, L2.2, U$1.VIN; no longer C5.1, C6.1, L3.2, U$2.VIN
- net N$55: now also R109.1; no longer R58.1
- net N$56: now also R114.2; no longer R8.2
- net N$6: now also C2.1, L1.2, L2.1; no longer C3.1, L2.2, L3.1
- net N$67: now also BAR.C, R143.2; no longer BAR.A, R70.2
- net N$68: now also IC101.GPB5; no longer R21.2
- net N$69: now also BEAT.C, R144.2; no longer BAR.C, IC2.GPB4
- net N$7: now also C10.2, U$1.BST; no longer C8.2, U$2.BST
- net N$71: now also R8.1; no longer R55.1
- net N$78: now also R9.2; no longer R54.2
- net N$8: now also C10.1, D3.C, L3.1, U$1.SW; no longer C8.1, D1.C, L1.1, U$2.SW
- net N$86: now also C17.2, C19.1, C27.2, U1.LDO_OUT; no longer C14.2, C15.2
- net N$9: now also C11.1, U$1.FB; no longer C9.1, U$2.FB
- net RUN: now also J1.10; no longer PL1.10
- net SWCLK: now also J1.4; no longer PL1.4
- net SWDI0: now also J1.2; no longer PL1.2
- net VCC: now also C13.+, C14.1, C15.1, C18.2, C20.1, C21.1, C22.2, C23.2, C24.2, C25.2, C26.2, J1.1, R5.2, U$2.VCC; no longer C11.+, C13.1, C17.1, C42.1, C43.1, C44.2, C45.2, C46.2, C47.2, C48.2, C49.2, C51.2, PL1.1, R6.2, U$1.VCC
Other:
- moved on the sheet: +*-, BAR, BEAT, C10, C12, C14, C15, C16, C17, C19, C21, C22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
